File: kicad/interface.sch (KiCad schematic (older format))
At the start: 0 parts

Commit message: add components to library. start electric schematic
Parts:
- added J?: Conn_02x20_Odd_Even, symbol Conn_02x20_Odd_Even
Changed lines of the file:
@@
 $Descr A4 11693 8268
 encoding utf-8
-Sheet 1 4
+Sheet 2 4
 Title ""
 Date ""
@@
 Comment4 ""
 $EndDescr
-$Sheet
-S 1800 1400 2200 1550
-U 5AC7805B
-F0 "interface" 60
-F1 "interface.sch" 60
-$EndSheet
-$Sheet
-S 5100 1400 2200 1550
-U 5AC7807D
-F0 "ethernet" 60
-F1 "ethernet.sch" 60
-$EndSheet
-$Sheet
-S 3800 3500 2550 1800
-U 5AC78096
-F0 "power" 60
-F1 "power.sch" 60
-$EndSheet
+$Comp
+L Conn_02x20_Odd_Even J?
+U 1 1 5AC78E04
+P 1800 2200
+F 0 "J?" H 1850 3200 50  0000 C CNN
+F 1 "Conn_02x20_Odd_Even" H 1850 1100 50  0000 C CNN
+F 2 "" H 1800 2200 50  0001 C CNN
+F 3 "" H 1800 2200 50  0001 C CNN
+	1    1800 2200
+	1    0    0    -1
+$EndComp
 $EndSCHEMATC

Commit message: add ksz9021gn, cfps-73 to library
Parts:
- added D? (x5): 10cl025, symbol 10cl025
- added D?: NUP4114UPXV6T1G, symbol NUP4114UPXV6T1G
- added G?: CFPS-73, symbol CFPS-73
- added J? (x2): Conn_02x05_Odd_Even, symbol Conn_02x05_Odd_Even
- added U?: 24LC32, Housings_SOIC:SOIC-8_3.9x4.9mm_Pitch1.27mm, symbol 24LC32
Other:
- moved on the sheet: J?
Changed lines of the file:
@@
 LIBS:contrib
 LIBS:valves
-LIBS:88e1512
 LIBS:10cl025
 LIBS:l829-1j1t-43
 LIBS:nup4114upxv6t1g
+LIBS:ksz9021rl
+LIBS:ksz9021gn
+LIBS:cfps-73
+LIBS:fpgagigepi-cache
 EELAYER 25 0
 EELAYER END
@@
 encoding utf-8
 Sheet 2 4
-Title ""
-Date ""
-Rev ""
-Comp ""
-Comment1 ""
-Comment2 ""
+Title "figa-pi"
+Date "2018-04-13"
+Rev "1.0"
+Comp "GENERAL RND"
+Comment1 "07e20003"
+Comment2 "Y. Remizov"
 Comment3 ""
 Comment4 ""
@@
 L Conn_02x20_Odd_Even J?
 U 1 1 5AC78E04
-P 1800 2200
-F 0 "J?" H 1850 3200 50  0000 C CNN
-F 1 "Conn_02x20_Odd_Even" H 1850 1100 50  0000 C CNN
-F 2 "" H 1800 2200 50  0001 C CNN
-F 3 "" H 1800 2200 50  0001 C CNN
-	1    1800 2200
+P 4700 2200
+F 0 "J?" H 4750 3200 50  0000 C CNN
+F 1 "Conn_02x20_Odd_Even" H 4750 1100 50  0000 C CNN
+F 2 "" H 4700 2200 50  0001 C CNN
+F 3 "" H 4700 2200 50  0001 C CNN
+	1    4700 2200
 	1    0    0    -1
 $EndComp
+$Comp
+L 10cl025 D?
+U 1 1 5AD09E19
+P 8550 2000
+F 0 "D?" H 8200 2950 60  0000 C CNN
+F 1 "10cl025" H 8750 2950 60  0000 C CNN
+F 2 "" H 7550 2350 60  0001 C CNN
+F 3 "" H 7550 2350 60  0001 C CNN
+	1    8550 2000
+	1    0    0    -1
+$EndComp
+$Comp
+L 10cl025 D?
+U 2 1 5AD09EC2
+P 8550 3700
+F 0 "D?" H 8200 4150 60  0000 C CNN
+F 1 "10cl025" H 8800 4150 60  0000 C CNN
+F 2 "" H 7550 4050 60  0001 C CNN
+F 3 "" H 7550 4050 60  0001 C CNN
+	2    8550 3700
+	1    0    0    -1
+$EndComp
+$Comp
+L 10cl025 D?
+U 3 1 5AD09F07
+P 10150 1600
+F 0 "D?" H 9800 2150 60  0000 C CNN
+F 1 "10cl025" H 10400 2150 60  0000 C CNN
+F 2 "" H 9150 1950 60  0001 C CNN
+F 3 "" H 9150 1950 60  0001 C CNN
+	3    10150 1600
+	1    0    0    -1
+$EndComp
+$Comp
+L 10cl025 D?
+U 5 1 5AD09F80
+P 10150 3000
+F 0 "D?" H 9800 3550 60  0000 C CNN
+F 1 "10cl025" H 10400 3550 60  0000 C CNN
+F 2 "" H 9150 3350 60  0001 C CNN
+F 3 "" H 9150 3350 60  0001 C CNN
+	5    10150 3000
+	1    0    0    -1
+$EndComp
+$Comp
+L 10cl025 D?
+U 6 1 5AD09FE7
+P 10150 4800
+F 0 "D?" H 9800 5750 60  0000 C CNN
+F 1 "10cl025" H 10350 5750 60  0000 C CNN
+F 2 "" H 9150 5150 60  0001 C CNN
+F 3 "" H 9150 5150 60  0001 C CNN
+	6    10150 4800
+	1    0    0    -1
+$EndComp
+$Comp
+L Conn_02x05_Odd_Even J?
+U 1 1 5AD0A09E
+P 1750 3950
+F 0 "J?" H 1800 4250 50  0000 C CNN
+F 1 "Conn_02x05_Odd_Even" H 1800 3650 50  0000 C CNN
+F 2 "" H 1750 3950 50  0001 C CNN
+F 3 "" H 1750 3950 50  0001 C CNN
+	1    1750 3950
+	1    0    0    -1
+$EndComp
+$Comp
+L 24LC32 U?
+U 1 1 5AD0A4F1
+P 1800 7200
+F 0 "U?" H 1550 7450 50  0000 C CNN
+F 1 "24LC32" H 1850 7450 50  0000 L CNN
+F 2 "Housings_SOIC:SOIC-8_3.9x4.9mm_Pitch1.27mm" H 1850 6950 50  0001 L CNN
+F 3 "" H 1800 7100 50  0001 C CNN
+	1    1800 7200
+	1    0    0    -1
+$EndComp
+$Comp
+L Conn_02x05_Odd_Even J?
+U 1 1 5AD0A849
+P 6550 2600
+F 0 "J?" H 6600 2900 50  0000 C CNN
+F 1 "Conn_02x05_Odd_Even" H 6600 2300 50  0000 C CNN
+F 2 "" H 6550 2600 50  0001 C CNN
+F 3 "" H 6550 2600 50  0001 C CNN
+	1    6550 2600
+	1    0    0    -1
+$EndComp
+$Comp
+L NUP4114UPXV6T1G D?
+U 1 1 5AD0A880
+P 6650 3500
+F 0 "D?" H 6450 3800 60  0000 C CNN
+F 1 "NUP4114UPXV6T1G" H 6650 3200 60  0000 C CNN
+F 2 "" H 6650 3450 60  0001 C CNN
+F 3 "" H 6650 3450 60  0001 C CNN
+	1    6650 3500
+	1    0    0    -1
+$EndComp
+$Comp
+L CFPS-73 G?
+U 1 1 5AD09F7E
+P 1700 6300
+F 0 "G?" H 1550 6550 60  0000 C CNN
+F 1 "CFPS-73" H 1700 6050 60  0000 C CNN
+F 2 "" H 1700 6300 60  0001 C CNN
+F 3 "" H 1700 6300 60  0001 C CNN
+	1    1700 6300
+	1    0    0    -1
+$EndComp

Commit message: add tlv62080 to library, continue design schematic
Parts:
- added C5: 0.1, symbol C
- added C6: C, symbol C
- added J7: Conn_01x02, symbol Conn_01x02
- added R1, R2: 3.9k, symbol R
- added R3, R6: 1k, symbol R
- added R4, R5: 10k, symbol R
- gave numbers to parts that had none: 7
Connections:
- net GND: now reaches J2.14 (Pin_14)
- net GND: now also D1.2 (Vn), G1.2 (GND), J2.20 (Pin_20), J2.25 (Pin_25), J2.30 (Pin_30), J2.34 (Pin_34), J2.39 (Pin_39), J2.6 (Pin_6), J2.9 (Pin_9), J3.10 (Pin_10), J3.2 (Pin_2), U1.1 (A0), U1.2 (A1), U1.3 (A2), U1.4 (GND), C5.2, C6.2, J7.2 (Pin_2), R6.1
- net +5V: now reaches J2.2 (Pin_2)
- net +5V: now also J2.4 (Pin_4)
- net SDA: now reaches J2.3 (Pin_3)
- net SDA: now also U1.5 (SDA), R1.2
- net SCL: now reaches J2.5 (Pin_5)
- net SCL: now also U1.6 (SCL), R2.2
- net JTAG_TDI: now reaches D2.15 (TDI)
- net JTAG_TDI: now also D1.4 (I/O3), J3.9 (Pin_9), R4.2
- net JTAG_TCK: now reaches D2.16 (TCK)
- net JTAG_TCK: now also D1.6 (I/O4), J3.1 (Pin_1), R6.2
- net JTAG_TMS: now reaches D2.18 (TMS)
- net JTAG_TMS: now also D1.3 (I/O2), J3.5 (Pin_5), R5.2
- net JTAG_TDO: now reaches D2.20 (TDO)
- net JTAG_TDO: now also D1.1 (I/O1), J3.3 (Pin_3)
- net 25MHz: now reaches G1.3 (OUT)
- net +3V3: now reaches G1.4 (Vdd)
- net +3V3: now also D1.5 (Vp), J3.4 (Pin_4), U1.8 (VCC), C5.1, C6.1, R1.1, R2.1, R3.1, R4.1, R5.1
- net at U1.7 (WP): now also J7.1 (Pin_1), R3.2
- no-connect marks 0 -> 42
Other:
- moved on the sheet: D1, G1, J1, J3, U1

Commit message: add nb3l553dr2g to library, continue design schematic
Parts:
- added C45: C, symbol C
- added D10, D11, D12: LED, symbol LED
- added D9: NB3L553, symbol NB3L553
- added R15, R16, R17: R, symbol R
Connections:
- net +3V3: now also C45.1, D9.1 (Vdd), D9.8 (OE), R15.2, R16.2, R17.2
- net GND: now also C45.2, D12.1 (K), D9.4 (GND)
- net USER_LED0: now reaches D2.10 (IO_10)
- net USER_LED0: now also D10.1 (K)
- net USER_LED1: now reaches D2.11 (IO_11)
- net USER_LED1: now also D11.1 (K)
- net 25MHz: no longer names the net of G1.3 (OUT)
- net 25MHz: now also D9.5 (Iclk)
- new net: D10.2 (A), R15.1
- new net: D12.2 (A), R17.1
- new net: D11.2 (A), R16.1
- new net 25M_A: D9.2 (Q0)
- new net 25M_B: D9.3 (Q1)
- no-connect marks 42 -> 44
Other:
- moved on the sheet: C6, G1

Commit message: continue design schematic
Parts:
- removed D1: NUP4114UPXV6T1G, symbol NUP4114UPXV6T1G
- removed D9: NB3L553, symbol NB3L553
- added D1: LED, symbol LED
- added R18, R19, R20: R, symbol R
- added U4: NUP4114UPXV6T1G, symbol NUP4114UPXV6T1G
- added U5: NB3L553, symbol NB3L553
Connections:
- net +3V3: now also R18.2, R19.2, R20.1, U4.5 (Vp), U5.1 (Vdd), U5.8 (OE)
- net 25M_A: now also U5.2 (Q0)
- net 25M_B: now also U5.3 (Q1)
- net GND: now also D2.21 (nCE), D2.22 (CLK0), D2.23 (CLK1), D2.90 (CLK5), D2.91 (CLK4), U4.2 (Vn), U5.4 (GND)
- net JTAG_TCK: now also U4.6 (I/O4)
- net JTAG_TDI: now also U4.4 (I/O3)
- net JTAG_TDO: now also U4.1 (I/O1)
- net JTAG_TMS: now also U4.3 (I/O2)
- net CONF_DONE: now reaches J2.11 (Pin_11)
- net CONF_DONE: now also D2.92 (CONF_DONE), D1.1 (K), R20.2
- net nSTATUS: now reaches J2.13 (Pin_13)
- net nSTATUS: now also D2.9 (nSTATUS), R19.1
- net nCONFIG: now reaches J2.15 (Pin_15)
- net nCONFIG: now also D2.14 (nCONFIG)
- net DATA: now reaches J2.19 (Pin_19)
- net DATA: now also D2.13 (IO_13/DATA0)
- net DCLK: now reaches J2.23 (Pin_23)
- net DCLK: now also D2.12 (IO_12/DCLK)
- net at G1.3 (OUT): now also U5.5 (Iclk)
- new net: D1.2 (A), R18.1
- no-connect marks 44 -> 39
Other:
- note added: "TODO\n-msel to config\n- gpio fpga to J1\n- gpio fpga to rPI\n- ext leds?\n- nominal res and cap\n- check gpio"
- moved on the sheet: D2B, D2F

Commit message: finished electrical connections
Parts:
- added D4, D5: LED, symbol LED
- added R32, R33: R, symbol R
Connections:
- net +3V3: now also R32.2, R33.2
- net +5V: now also J1.1 (Pin_1)
- net GND: now also D2.24 (CLK2), D2.25 (CLK3), D2.52 (CLK15), D2.53 (CLK14), D2.88 (CLK7), D2.89 (CLK6), D2.94 (MSEL0), D2.96 (MSEL1), D2.97 (MSEL2), J1.9 (Pin_9)
- net UART0_RX: now reaches J2.10 (Pin_10)
- net UART0_RX: now also J1.10 (Pin_10)
- net IO_51: now reaches J2.12 (Pin_12)
- net IO_51: now also D2.51 (IO_51)
- net IO_6: now reaches J2.16 (Pin_16)
- net IO_6: now also D2.6 (IO_6/ASDO/DATA1)
- net IO_8: now reaches J2.18 (Pin_18)
- net IO_8: now also D2.8 (IO_8/FLS_nCE/nCSO)
- net IO_99: now reaches J2.21 (Pin_21)
- net IO_99: now also D2.99 (IO_99/CRC_ERROR)
- net IO_85: now reaches J2.22 (Pin_22)
- net IO_85: now also D2.85 (IO_85)
- net IO_86: now reaches J2.24 (Pin_24)
- net IO_86: now also D2.86 (IO_86/DEV_OE)
- net IO_87: now reaches J2.26 (Pin_26)
- net IO_87: now also D2.87 (IO_87/DEV_CLRn)
- net IO_76: now reaches J2.29 (Pin_29)
- net IO_76: now also D2.76 (IO_76)
- net IO_77: now reaches J2.31 (Pin_31)
- net IO_77: now also D2.77 (IO_77)
- net IO_98: now reaches J2.32 (Pin_32)
- net IO_98: now also D2.98 (IO_98/INIT_DONE)
- net IO_80: now reaches J2.33 (Pin_33)
- net IO_80: now also D2.80 (IO_80)
- net PI_GPIO19/SPI1_MISO: now reaches J2.35 (Pin_35)
- net PI_GPIO19/SPI1_MISO: now also D2.28 (IO_28)
- net PI_GPIO16/SPI1_CS0: now reaches J2.36 (Pin_36)
- net PI_GPIO16/SPI1_CS0: now also D2.33 (IO_33)
- net IO_83: now reaches J2.37 (Pin_37)
- net IO_83: now also D2.83 (IO_83)
- net PI_GPIO20/SPI1_MOSI: now reaches J2.38 (Pin_38)
- net PI_GPIO20/SPI1_MOSI: now also D2.31 (IO_31)
- net PI_GPIO21/SPI1_SCLK: now reaches J2.40 (Pin_40)
- net PI_GPIO21/SPI1_SCLK: now also D2.32 (IO_32)
- net IO_50: now reaches J2.7 (Pin_7)
- net IO_50: now also D2.50 (IO_50)
- net UART0_TX: now reaches J2.8 (Pin_8)
- net UART0_TX: now also J1.8 (Pin_8)
- net INT_N: now reaches D2.7 (IO_7)
- net IO_39: now reaches D2.39 (IO_39)
- net IO_39: now also J1.3 (Pin_3)
- net IO_42: now reaches D2.42 (IO_42)
- net IO_42: now also J1.5 (Pin_5)
- net IO_43: now reaches D2.43 (IO_43)
- net IO_43: now also J1.7 (Pin_7)
- net IO_44: now reaches D2.44 (IO_44)
- net IO_44: now also J1.2 (Pin_2)
- net IO_46: now reaches D2.46 (IO_46)
- net IO_46: now also J1.4 (Pin_4)
- net IO_49: now reaches D2.49 (IO_49)
- net IO_49: now also J1.6 (Pin_6)
- net USER_LED2: now reaches D2.105 (IO_105)
- net USER_LED2: now also D4.1 (K)
- net USER_LED3: now reaches D2.106 (IO_106)
- net USER_LED3: now also D5.1 (K)
- new net: D4.2 (A), R32.1
- new net: D5.2 (A), R33.1
- no-connect marks 39 -> 13
Other:
- note added: "0,0,0 - PS, standart"
- note added: "TODO\n- nominal res and cap\n- nSTATUS opendrain\n- arrows"
- note removed: "TODO\n-msel to config\n- gpio fpga to J1\n- gpio fpga to rPI\n- ext leds?\n- nominal res and cap\n- check gpio"
- moved on the sheet: C5, D1, D10, D11, D2A, D2B, D2C, D2E, D2F, J1, J2, J3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

Commit message: write nominal of components
Parts:
- C45, C6: value C -> 0.1u
- C5: value 0.1 -> 0.1u
- R1, R2, R3, R4, R5, R6: footprint (none) -> Resistors_SMD:R_0603_HandSoldering
- R15, R16, R17, R18, R32, R33: value R -> 390; footprint (none) -> Resistors_SMD:R_0603_HandSoldering
- R19, R20: value R -> 10k; footprint (none) -> Resistors_SMD:R_0603_HandSoldering
Other:
- note removed: "TODO\n- nominal res and cap\n- nSTATUS opendrain\n- arrows"
Changed lines of the file:
@@
 F 0 "R1" V 2380 1100 50  0000 C CNN
 F 1 "3.9k" V 2300 1100 50  0000 C CNN
-F 2 "" V 2230 1100 50  0001 C CNN
+F 2 "Resistors_SMD:R_0603_HandSoldering" V 2230 1100 50  0001 C CNN
 F 3 "" H 2300 1100 50  0001 C CNN
 	1    2300 1100
@@
 F 0 "R2" V 2530 1100 50  0000 C CNN
 F 1 "3.9k" V 2450 1100 50  0000 C CNN
-F 2 "" V 2380 1100 50  0001 C CNN
+F 2 "Resistors_SMD:R_0603_HandSoldering" V 2380 1100 50  0001 C CNN
 F 3 "" H 2450 1100 50  0001 C CNN
 	1    2450 1100
@@
 F 0 "R3" V 2680 1100 50  0000 C CNN
 F 1 "1k" V 2600 1100 50  0000 C CNN
-F 2 "" V 2530 1100 50  0001 C CNN
+F 2 "Resistors_SMD:R_0603_HandSoldering" V 2530 1100 50  0001 C CNN
 F 3 "" H 2600 1100 50  0001 C CNN
 	1    2600 1100
@@
 P 1300 1100
 F 0 "C5" H 1325 1200 50  0000 L CNN
-F 1 "0.1" H 1325 1000 50  0000 L CNN
+F 1 "0.1u" H 1325 1000 50  0000 L CNN
 F 2 "" H 1338 950 50  0001 C CNN
 F 3 "" H 1300 1100 50  0001 C CNN
@@
 F 0 "R4" V 1580 2700 50  0000 C CNN
 F 1 "10k" V 1500 2700 50  0000 C CNN
-F 2 "" V 1430 2700 50  0001 C CNN
+F 2 "Resistors_SMD:R_0603_HandSoldering" V 1430 2700 50  0001 C CNN
 F 3 "" H 1500 2700 50  0001 C CNN
 	1    1500 2700
@@
 F 0 "R5" V 1780 2700 50  0000 C CNN
 F 1 "10k" V 1700 2700 50  0000 C CNN
-F 2 "" V 1630 2700 50  0001 C CNN
+F 2 "Resistors_SMD:R_0603_HandSoldering" V 1630 2700 50  0001 C CNN
 F 3 "" H 1700 2700 50  0001 C CNN
 	1    1700 2700
@@
 F 0 "R6" V 2230 4450 50  0000 C CNN
 F 1 "1k" V 2150 4450 50  0000 C CNN
-F 2 "" V 2080 4450 50  0001 C CNN
+F 2 "Resistors_SMD:R_0603_HandSoldering" V 2080 4450 50  0001 C CNN
 F 3 "" H 2150 4450 50  0001 C CNN
 	1    2150 4450
@@
 P 1100 6950
 F 0 "C6" H 1125 7050 50  0000 L CNN
-F 1 "C" H 1125 6850 50  0000 L CNN
+F 1 "0.1u" H 1125 6850 50  0000 L CNN
 F 2 "" H 1138 6800 50  0001 C CNN
 F 3 "" H 1100 6950 50  0001 C CNN
@@
 P 3050 6750
 F 0 "C45" H 3075 6850 50  0000 L CNN
-F 1 "C" H 3075 6650 50  0000 L CNN
+F 1 "0.1u" H 3075 6650 50  0000 L CNN
 F 2 "" H 3088 6600 50  0001 C CNN
 F 3 "" H 3050 6750 50  0001 C CNN
@@
 P 1350 5300
 F 0 "R15" V 1430 5300 50  0000 C CNN
-F 1 "R" V 1350 5300 50  0000 C CNN
-F 2 "" V 1280 5300 50  0001 C CNN
+F 1 "390" V 1350 5300 50  0000 C CNN
+F 2 "Resistors_SMD:R_0603_HandSoldering" V 1280 5300 50  0001 C CNN
 F 3 "" H 1350 5300 50  0001 C CNN
 	1    1350 5300
@@
 P 1350 5500
 F 0 "R16" V 1430 5500 50  0000 C CNN
-F 1 "R" V 1350 5500 50  0000 C CNN
-F 2 "" V 1280 5500 50  0001 C CNN
+F 1 "390" V 1350 5500 50  0000 C CNN
+F 2 "Resistors_SMD:R_0603_HandSoldering" V 1280 5500 50  0001 C CNN
 F 3 "" H 1350 5500 50  0001 C CNN
 	1    1350 5500
@@
 P 1350 6100
 F 0 "R17" V 1430 6100 50  0000 C CNN
-F 1 "R" V 1350 6100 50  0000 C CNN
-F 2 "" V 1280 6100 50  0001 C CNN
+F 1 "390" V 1350 6100 50  0000 C CNN
+F 2 "Resistors_SMD:R_0603_HandSoldering" V 1280 6100 50  0001 C CNN
 F 3 "" H 1350 6100 50  0001 C CNN
 	1    1350 6100
@@
 P 9450 950
 F 0 "R19" V 9530 950 50  0000 C CNN
-F 1 "R" V 9450 950 50  0000 C CNN
-F 2 "" V 9380 950 50  0001 C CNN
+F 1 "10k" V 9450 950 50  0000 C CNN
+F 2 "Resistors_SMD:R_0603_HandSoldering" V 9380 950 50  0001 C CNN
 F 3 "" H 9450 950 50  0001 C CNN
 	1    9450 950
@@
 P 9500 3350
 F 0 "R20" V 9580 3350 50  0000 C CNN
-F 1 "R" V 9500 3350 50  0000 C CNN
-F 2 "" V 9430 3350 50  0001 C CNN
+F 1 "10k" V 9500 3350 50  0000 C CNN
+F 2 "Resistors_SMD:R_0603_HandSoldering" V 9430 3350 50  0001 C CNN
 F 3 "" H 9500 3350 50  0001 C CNN
 	1    9500 3350
@@
 P 1350 5100
 F 0 "R18" V 1430 5100 50  0000 C CNN
-F 1 "R" V 1350 5100 50  0000 C CNN
-F 2 "" V 1280 5100 50  0001 C CNN
+F 1 "390" V 1350 5100 50  0000 C CNN
+F 2 "Resistors_SMD:R_0603_HandSoldering" V 1280 5100 50  0001 C CNN
 F 3 "" H 1350 5100 50  0001 C CNN
 	1    1350 5100
@@
 U 1 1 5AD8258F
 P 1850 5100
-F 0 "D1" H 1850 5200 50  0000 C CNN
-F 1 "LED" H 1850 5000 50  0000 C CNN
+F 0 "D1" H 2000 5150 50  0000 C CNN
+F 1 "LED" H 1700 5150 50  0000 C CNN
 F 2 "" H 1850 5100 50  0001 C CNN
 F 3 "" H 1850 5100 50  0001 C CNN
@@
 Text GLabel 6000 1600 0    60   Input ~ 0
 CONF_DONE
-Text Notes 8100 7050 0    60   ~ 0
-TODO\n- nominal res and cap\n- nSTATUS opendrain\n- arrows
 Wire Wire Line
 	6800 1000 6800 1200
@@
 P 1350 5700
 F 0 "R32" V 1430 5700 50  0000 C CNN
-F 1 "R" V 1350 5700 50  0000 C CNN
-F 2 "" V 1280 5700 50  0001 C CNN
+F 1 "390" V 1350 5700 50  0000 C CNN
+F 2 "Resistors_SMD:R_0603_HandSoldering" V 1280 5700 50  0001 C CNN
 F 3 "" H 1350 5700 50  0001 C CNN
 	1    1350 5700
@@
 P 1350 5900
 F 0 "R33" V 1430 5900 50  0000 C CNN
-F 1 "R" V 1350 5900 50  0000 C CNN
-F 2 "" V 1280 5900 50  0001 C CNN
+F 1 "390" V 1350 5900 50  0000 C CNN
+F 2 "Resistors_SMD:R_0603_HandSoldering" V 1280 5900 50  0001 C CNN
 F 3 "" H 1350 5900 50  0001 C CNN
 	1    1350 5900

Commit message: place components to pcb, add footprints of cfps-73 l829 sot-563
Parts:
- C45, C5, C6: footprint (none) -> Capacitors_SMD:C_0603_HandSoldering
- D1, D10, D11, D12, D4, D5: footprint (none) -> LEDs:LED_0603_HandSoldering
- G1: footprint (none) -> library:CFPS-73
- J1, J3: footprint (none) -> Pin_Headers:Pin_Header_Straight_2x05_Pitch2.54mm
- J2: footprint (none) -> Pin_Headers:Pin_Header_Straight_2x20_Pitch2.54mm
- J7: footprint (none) -> Pin_Headers:Pin_Header_Straight_1x02_Pitch2.54mm
- U4: footprint (none) -> library:SOT-563-6
- U5: footprint (none) -> Housings_DFN_QFN:DFN-8-1EP_2x2mm_Pitch0.5mm
Connections:
- net GND: now also U5.9 (EXPPAD)
Changed lines of the file:
@@
 F 0 "J2" H 6450 3000 50  0000 C CNN
 F 1 "Conn_02x20_Odd_Even" H 6450 900 50  0000 C CNN
-F 2 "" H 6400 2000 50  0001 C CNN
+F 2 "Pin_Headers:Pin_Header_Straight_2x20_Pitch2.54mm" H 6400 2000 50  0001 C CNN
 F 3 "" H 6400 2000 50  0001 C CNN
 	1    6400 2000
@@
 F 0 "J1" H 8250 6100 50  0000 C CNN
 F 1 "Conn_02x05_Odd_Even" H 8250 5500 50  0000 C CNN
-F 2 "" H 8200 5800 50  0001 C CNN
+F 2 "Pin_Headers:Pin_Header_Straight_2x05_Pitch2.54mm" H 8200 5800 50  0001 C CNN
 F 3 "" H 8200 5800 50  0001 C CNN
 	1    8200 5800
@@
 F 0 "J3" H 2250 3450 50  0000 C CNN
 F 1 "Conn_02x05_Odd_Even" H 2250 2850 50  0000 C CNN
-F 2 "" H 2200 3150 50  0001 C CNN
+F 2 "Pin_Headers:Pin_Header_Straight_2x05_Pitch2.54mm" H 2200 3150 50  0001 C CNN
 F 3 "" H 2200 3150 50  0001 C CNN
 	1    2200 3150
@@
 F 0 "G1" H 1650 7200 60  0000 C CNN
 F 1 "CFPS-73" H 1800 6700 60  0000 C CNN
-F 2 "" H 1800 6950 60  0001 C CNN
+F 2 "library:CFPS-73" H 1800 6950 60  0001 C CNN
 F 3 "" H 1800 6950 60  0001 C CNN
 	1    1800 6950
@@
 F 0 "C5" H 1325 1200 50  0000 L CNN
 F 1 "0.1u" H 1325 1000 50  0000 L CNN
-F 2 "" H 1338 950 50  0001 C CNN
+F 2 "Capacitors_SMD:C_0603_HandSoldering" H 1338 950 50  0001 C CNN
 F 3 "" H 1300 1100 50  0001 C CNN
 	1    1300 1100
@@
 F 0 "J7" H 2800 1750 50  0000 C CNN
 F 1 "Conn_01x02" H 2800 1450 50  0000 C CNN
-F 2 "" H 2800 1650 50  0001 C CNN
+F 2 "Pin_Headers:Pin_Header_Straight_1x02_Pitch2.54mm" H 2800 1650 50  0001 C CNN
 F 3 "" H 2800 1650 50  0001 C CNN
 	1    2800 1650
@@
 F 0 "C6" H 1125 7050 50  0000 L CNN
 F 1 "0.1u" H 1125 6850 50  0000 L CNN
-F 2 "" H 1138 6800 50  0001 C CNN
+F 2 "Capacitors_SMD:C_0603_HandSoldering" H 1138 6800 50  0001 C CNN
 F 3 "" H 1100 6950 50  0001 C CNN
 	1    1100 6950
@@
 F 0 "C45" H 3075 6850 50  0000 L CNN
 F 1 "0.1u" H 3075 6650 50  0000 L CNN
-F 2 "" H 3088 6600 50  0001 C CNN
+F 2 "Capacitors_SMD:C_0603_HandSoldering" H 3088 6600 50  0001 C CNN
 F 3 "" H 3050 6750 50  0001 C CNN
 	1    3050 6750
@@
 L GND #PWR012
 U 1 1 5AD5DFDE
-P 3300 7250
-F 0 "#PWR012" H 3300 7000 50  0001 C CNN
-F 1 "GND" H 3300 7100 50  0000 C CNN
-F 2 "" H 3300 7250 50  0001 C CNN
-F 3 "" H 3300 7250 50  0001 C CNN
-	1    3300 7250
-	1    0    0    -1
+P 3250 7550
+F 0 "#PWR012" H 3250 7300 50  0001 C CNN
+F 1 "GND" H 3250 7400 50  0000 C CNN
+F 2 "" H 3250 7550 50  0001 C CNN
+F 3 "" H 3250 7550 50  0001 C CNN
+	1    3250 7550
+	0    1    1    0
 $EndComp
 $Comp
@@
 F 0 "D10" H 2000 5350 50  0000 C CNN
 F 1 "LED" H 1700 5350 50  0000 C CNN
-F 2 "" H 1850 5300 50  0001 C CNN
+F 2 "LEDs:LED_0603_HandSoldering" H 1850 5300 50  0001 C CNN
 F 3 "" H 1850 5300 50  0001 C CNN
 	1    1850 5300
@@
 F 0 "D12" H 2000 6150 50  0000 C CNN
 F 1 "LED" H 1700 6150 50  0000 C CNN
-F 2 "" H 1850 6100 50  0001 C CNN
+F 2 "LEDs:LED_0603_HandSoldering" H 1850 6100 50  0001 C CNN
 F 3 "" H 1850 6100 50  0001 C CNN
 	1    1850 6100
@@
 F 0 "D11" H 2000 5550 50  0000 C CNN
 F 1 "LED" H 1700 5550 50  0000 C CNN
-F 2 "" H 1850 5500 50  0001 C CNN
+F 2 "LEDs:LED_0603_HandSoldering" H 1850 5500 50  0001 C CNN
 F 3 "" H 1850 5500 50  0001 C CNN
 	1    1850 5500
@@
 	3400 7150 3300 7150
 Wire Wire Line
-	3300 7150 3300 7250
-Wire Wire Line
 	3400 7050 2400 7050
 Wire Wire Line
@@
 F 0 "U4" H 2250 4300 60  0000 C CNN
 F 1 "NUP4114UPXV6T1G" H 2450 3700 60  0000 C CNN
-F 2 "" H 2450 3950 60  0001 C CNN
+F 2 "library:SOT-563-6" H 2450 3950 60  0001 C CNN
 F 3 "" H 2450 3950 60  0001 C CNN
 	1    2450 4000
@@
 P 3800 6950
 F 0 "U5" H 3650 7300 60  0000 C CNN
-F 1 "NB3L553" H 3800 6600 60  0000 C CNN
-F 2 "" H 3800 6950 60  0001 C CNN
+F 1 "NB3L553" H 4050 6550 60  0000 C CNN
+F 2 "Housings_DFN_QFN:DFN-8-1EP_2x2mm_Pitch0.5mm" H 3800 6950 60  0001 C CNN
 F 3 "" H 3800 6950 60  0001 C CNN
 	1    3800 6950
@@
 F 0 "D1" H 2000 5150 50  0000 C CNN
 F 1 "LED" H 1700 5150 50  0000 C CNN
-F 2 "" H 1850 5100 50  0001 C CNN
+F 2 "LEDs:LED_0603_HandSoldering" H 1850 5100 50  0001 C CNN
 F 3 "" H 1850 5100 50  0001 C CNN
 	1    1850 5100
@@
 F 0 "D4" H 2000 5750 50  0000 C CNN
 F 1 "LED" H 1700 5750 50  0000 C CNN
-F 2 "" H 1850 5700 50  0001 C CNN
+F 2 "LEDs:LED_0603_HandSoldering" H 1850 5700 50  0001 C CNN
 F 3 "" H 1850 5700 50  0001 C CNN
 	1    1850 5700
@@
 F 0 "D5" H 2000 5950 50  0000 C CNN
 F 1 "LED" H 1700 5950 50  0000 C CNN
-F 2 "" H 1850 5900 50  0001 C CNN
+F 2 "LEDs:LED_0603_HandSoldering" H 1850 5900 50  0001 C CNN
 F 3 "" H 1850 5900 50  0001 C CNN
 	1    1850 5900
@@
 Wire Wire Line
 	9800 4600 9300 4600
+Wire Wire Line
+	3250 7550 3800 7550
+Wire Wire Line
+	3300 7150 3300 7550
+Wire Wire Line
+	3800 7550 3800 7500
+Connection ~ 3300 7550
 $EndSCHEMATC
