File: kicad/fpgagigepi.sch (KiCad schematic (older format))
At the start: 0 parts

Commit message: add tlv62080 to library, continue design schematic
Changed lines of the file:
@@
 LIBS:ksz9021gn
 LIBS:cfps-73
+LIBS:tlv62080
 LIBS:fpgagigepi-cache
 EELAYER 25 0
@@
 $EndDescr
 $Sheet
-S 1800 1400 2200 1550
+S 1600 1400 2200 1550
 U 5AC7805B
 F0 "interface" 60

Commit message: Project translated to template "Raspberry Pi HAT" Added library files from template. Renamed refdes. Changed placement for all components
Parts:
- added H1, H2, H3, H4: 3mm_Mounting_Hole, project_footprints:NPTH_3mm_ID, symbol Mechanical:Mounting_Hole
Other:
- note added: "Mounting Holes"
Changed lines of the file:
@@
 EESchema Schematic File Version 2
+LIBS:74xgxx
+LIBS:74xx
+LIBS:ac-dc
+LIBS:actel
+LIBS:adc-dac
+LIBS:allegro
+LIBS:Altera
+LIBS:analog_devices
+LIBS:analog_switches
+LIBS:atmel
+LIBS:audio
+LIBS:battery_management
+LIBS:bbd
+LIBS:bosch
+LIBS:brooktre
+LIBS:cmos_ieee
+LIBS:cmos4000
+LIBS:conn
+LIBS:contrib
+LIBS:cypress
+LIBS:dc-dc
+LIBS:device
+LIBS:digital-audio
+LIBS:diode
+LIBS:display
+LIBS:dsp
+LIBS:elec-unifil
+LIBS:ESD_Protection
+LIBS:ftdi
+LIBS:gennum
+LIBS:graphic_symbols
+LIBS:hc11
+LIBS:infineon
+LIBS:intel
+LIBS:interface
+LIBS:intersil
+LIBS:ir
+LIBS:Lattice
+LIBS:leds
+LIBS:LEM
+LIBS:linear
+LIBS:logic_programmable
+LIBS:maxim
+LIBS:mechanical
+LIBS:memory
+LIBS:microchip
+LIBS:microchip_dspic33dsc
+LIBS:microchip_pic10mcu
+LIBS:microchip_pic12mcu
+LIBS:microchip_pic16mcu
+LIBS:microchip_pic18mcu
+LIBS:microchip_pic24mcu
+LIBS:microchip_pic32mcu
+LIBS:microcontrollers
+LIBS:modules
+LIBS:motor_drivers
+LIBS:motorola
+LIBS:motors
+LIBS:msp430
+LIBS:nordicsemi
+LIBS:nxp
+LIBS:nxp_armmcu
+LIBS:onsemi
+LIBS:opto
+LIBS:Oscillators
+LIBS:philips
 LIBS:power
-LIBS:device
+LIBS:Power_Management
+LIBS:powerint
+LIBS:pspice
+LIBS:references
+LIBS:regul
+LIBS:relays
+LIBS:rfcom
+LIBS:RFSolutions
+LIBS:sensors
+LIBS:silabs
+LIBS:siliconi
+LIBS:stm8
+LIBS:stm32
+LIBS:supertex
 LIBS:switches
-LIBS:relays
-LIBS:motors
+LIBS:texas
+LIBS:transf
 LIBS:transistors
-LIBS:conn
-LIBS:linear
-LIBS:regul
-LIBS:74xx
-LIBS:cmos4000
-LIBS:adc-dac
-LIBS:memory
+LIBS:triac_thyristor
+LIBS:ttl_ieee
+LIBS:valves
+LIBS:video
+LIBS:wiznet
+LIBS:Worldsemi
+LIBS:Xicor
 LIBS:xilinx
-LIBS:microcontrollers
-LIBS:dsp
-LIBS:microchip
-LIBS:analog_switches
-LIBS:motorola
-LIBS:texas
-LIBS:intel
-LIBS:audio
-LIBS:interface
-LIBS:digital-audio
-LIBS:philips
-LIBS:display
-LIBS:cypress
-LIBS:siliconi
-LIBS:opto
-LIBS:atmel
-LIBS:contrib
-LIBS:valves
+LIBS:zetex
+LIBS:Zilog
 LIBS:10cl025
+LIBS:88e1512
+LIBS:cfps-73
+LIBS:ksz9021gn
+LIBS:ksz9021rl
 LIBS:l829-1j1t-43
+LIBS:my
+LIBS:nb3l553
 LIBS:nup4114upxv6t1g
-LIBS:ksz9021rl
-LIBS:ksz9021gn
-LIBS:cfps-73
 LIBS:tlv62080
-LIBS:nb3l553
 LIBS:fpgagigepi-cache
 EELAYER 25 0
 EELAYER END
-$Descr A4 11693 8268
+$Descr A3 16535 11693
 encoding utf-8
 Sheet 1 4
-Title "figa-pi"
-Date "2018-04-13"
-Rev "1.0"
-Comp "GENERAL RND"
-Comment1 "07e20003"
-Comment2 "Y. Remizov"
+Title "Raspberry Pi HAT"
+Date ""
+Rev "A"
+Comp ""
+Comment1 ""
+Comment2 ""
 Comment3 ""
 Comment4 ""
 $EndDescr
+$Comp
+L Mechanical:Mounting_Hole H1
+U 1 1 5834BC4A
+P 1950 6250
+F 0 "H1" H 1800 6350 60  0000 C CNN
+F 1 "3mm_Mounting_Hole" H 1950 6100 60  0000 C CNN
+F 2 "project_footprints:NPTH_3mm_ID" H 1850 6250 60  0001 C CNN
+F 3 "" H 1850 6250 60  0001 C CNN
+F 4 "" H -16300 -4400 50  0001 C CNN "MFR"
+F 5 "" H -16300 -4400 50  0001 C CNN "MPN"
+F 6 "" H -16300 -4400 50  0001 C CNN "SPR"
+F 7 "" H -16300 -4400 50  0001 C CNN "SPN"
+F 8 "" H -16300 -4400 50  0001 C CNN "SPURL"
+	1    1950 6250
+	1    0    0    -1
+$EndComp
+$Comp
+L Mechanical:Mounting_Hole H3
+U 1 1 5834BCDF
+P 2950 6250
+F 0 "H3" H 2800 6350 60  0000 C CNN
+F 1 "3mm_Mounting_Hole" H 2950 6100 60  0000 C CNN
+F 2 "project_footprints:NPTH_3mm_ID" H 2850 6250 60  0001 C CNN
+F 3 "" H 2850 6250 60  0001 C CNN
+F 4 "" H -16300 -4400 50  0001 C CNN "MFR"
+F 5 "" H -16300 -4400 50  0001 C CNN "MPN"
+F 6 "" H -16300 -4400 50  0001 C CNN "SPR"
+F 7 "" H -16300 -4400 50  0001 C CNN "SPN"
+F 8 "" H -16300 -4400 50  0001 C CNN "SPURL"
+	1    2950 6250
+	1    0    0    -1
+$EndComp
+$Comp
+L Mechanical:Mounting_Hole H2
+U 1 1 5834BD62
+P 1950 6800
+F 0 "H2" H 1800 6900 60  0000 C CNN
+F 1 "3mm_Mounting_Hole" H 1950 6650 60  0000 C CNN
+F 2 "project_footprints:NPTH_3mm_ID" H 1850 6800 60  0001 C CNN
+F 3 "" H 1850 6800 60  0001 C CNN
+F 4 "" H -16300 -4400 50  0001 C CNN "MFR"
+F 5 "" H -16300 -4400 50  0001 C CNN "MPN"
+F 6 "" H -16300 -4400 50  0001 C CNN "SPR"
+F 7 "" H -16300 -4400 50  0001 C CNN "SPN"
+F 8 "" H -16300 -4400 50  0001 C CNN "SPURL"
+	1    1950 6800
+	1    0    0    -1
+$EndComp
+$Comp
+L Mechanical:Mounting_Hole H4
+U 1 1 5834BDED
+P 3000 6800
+F 0 "H4" H 2850 6900 60  0000 C CNN
+F 1 "3mm_Mounting_Hole" H 3000 6650 60  0000 C CNN
+F 2 "project_footprints:NPTH_3mm_ID" H 2900 6800 60  0001 C CNN
+F 3 "" H 2900 6800 60  0001 C CNN
+F 4 "" H -16300 -4400 50  0001 C CNN "MFR"
+F 5 "" H -16300 -4400 50  0001 C CNN "MPN"
+F 6 "" H -16300 -4400 50  0001 C CNN "SPR"
+F 7 "" H -16300 -4400 50  0001 C CNN "SPN"
+F 8 "" H -16300 -4400 50  0001 C CNN "SPURL"
+	1    3000 6800
+	1    0    0    -1
+$EndComp
+Text Notes 1600 5950 0    118  ~ 24
+Mounting Holes
 $Sheet
-S 1600 1400 2200 1550
-U 5AC7805B
-F0 "interface" 60
+S 4050 2050 3300 1500
+U 5B0D73F1
+F0 "interface.sch" 60
 F1 "interface.sch" 60
 $EndSheet
 $Sheet
-S 5100 1400 2200 1550
-U 5AC7807D
-F0 "ethernet" 60
+S 8150 2050 4200 1500
+U 5B0D756D
+F0 "ethernet.sch" 60
 F1 "ethernet.sch" 60
 $EndSheet
 $Sheet
-S 3800 3500 2550 1800
-U 5AC78096
-F0 "power" 60
+S 6700 4650 3950 1650
+U 5B0DA588
+F0 "power.sch" 60
 F1 "power.sch" 60
 $EndSheet
